File: KicadProjects/regulator_daughter_board/regulator_daughter_board.kicad_sch (KiCad schematic)
At the start: 7 parts, among them J1 Conn_01x04, U1 TPS613222ADBVR

Commit message: yup
Parts:
- J1: footprint Connector_PinSocket_1.00mm:PinSocket_1x04_P1.00mm_Vertical -> Connector_PinHeader_2.54mm:PinHeader_1x04_P2.54mm_Vertical
Changed lines of the file:
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@@
 			)
 		)
-		(property "Footprint" "Connector_PinSocket_1.00mm:PinSocket_1x04_P1.00mm_Vertical"
+		(property "Footprint" "Connector_PinHeader_2.54mm:PinHeader_1x04_P2.54mm_Vertical"
 			(at 124.46 106.68 0)
 			(effects
