File: KicadProjects/main_pcb/main_pcb.kicad_pcb (KiCad board)
At the start: 2 copper layers, 19 parts, among them SW1 09.03201.02, U1 MSP430G2553IPW20R

Commit message: yup
Parts:
- moved Sensor1 38.7 mm to (129.5, 128.6)
- moved LCD 15.6 mm to (157.5, 127.9)
- moved 3.3V1 13.6 mm to (117.3, 84.3)
- moved 5V1 13.6 mm to (117.3, 64.5)
- moved 10k 10.2 mm to (139.5, 110.0)
- renumbered R5 to 10k, R6 to 10k, R4 to 1k, R1 to 1k, R2 to 1k, 3.3V to 3.3V1, R3 to 510, 5V to 5V1, MOSFET1 to MOSFET, Potent.1 to Potent., SW1 to SW
Connections:
- SW pad 2: unconnected-(SW1-Pad2) -> Net-(3.3V1-Vin)
- SW pad 3: Net-(3.3V1-Vin) -> unconnected-(SW1-Pad3)
Routing:
- net Net-(Sensor1-Echo): track 35.0 -> 7.42 mm
- net Net-(5V1-Vout): track 82.1 -> 109.6 mm
- net Net-(3.3V1-Vin): track 35.3 -> 61.7 mm
- net Net-(Sensor1-Trg.): track 34.4 -> 11.1 mm
- net Net-(LCD1-SCL): track 10.0 -> 23.7 mm, vias 0 -> 1
- net Net-(LCD1-SDA): track 9.94 -> 22.9 mm, vias 0 -> 1
- net Net-(Programmer_Pins1-Reset): track 19.3 -> 25.5 mm
- net Net-(3.3V1-Vout): track 53.6 -> 56.8 mm
- net GNDPWR: vias 0 -> 3
- added copper zone on B.Cu, net GNDPWR
Other:
- board outline added: 88.8 x 106.6 mm
- board text added: "5V"
- board text added: "Ec."
- board text added: "LED"
- board text added: "SCL"
- board text added: "SDA"
- board text added: "Tr."
- board text added: "res."
- board text added: "test"

Commit message: main board finished
Parts:
- added REF**: charmander, footprints:charmander, F.Cu at (180.0, 125.0)
Routing:
- net GNDPWR: track 20.2 -> 15.8 mm
Other:
- board size 88.8 x 106.6 mm -> 88.8 x 99.1 mm
- board text added: "3.3V"
- board text added: "Yousef Alaa Awad"
